File: kicad/ratatech_echo/ratatech_echo.sch (KiCad schematic (older format))
At the start: 108 parts, among them J1 AudioJack2, J2 Conn_01x02, J3 Conn_01x02, J4 AudioJack2, J5 Barrel_Jack_Switch, Q1 2N3904, Q2 2N3906, Q3 2N3904, Q4 2N3906, SW1 SW_SPDT, SW2 SW_SPST, U1 NE5532, U2 NE5532, U3 PT2399, U4 LT1054xSOIC16, U5 LM7812_TO220, U6 LM7912_TO220

Commit message: Routing full done first try
Parts:
- removed C20: 560uF, Capacitor_SMD:C_0603_1608Metric, symbol Device:C
- removed SW1: SW_SPDT, Connector:FanPinHeader_1x03_P2.54mm_Vertical, symbol Switch:SW_SPDT
- added D9: LED, LED_SMD:LED_1206_3216Metric, symbol Device:LED
- added R39: 470, Resistor_SMD:R_0603_1608Metric, symbol Device:R
- added SW1: SW_DPDT_x2, M2028B2B1W03:M2028B2B1W03, symbol Switch:SW_DPDT_x2
Connections:
- net GND: now also D9.1 (K)
- net VCC: now also SW1.4 (A)
- net input: now also SW1.3 (C)
- net output: now also SW1.1 (A)
- net at J4.T: now also SW1.2 (B)
- new net: R39.2, SW1.5 (B)
- new net: D9.2 (A), R39.1
Other:
- moved on the sheet: C29
Changed lines of the file:
@@
 	20050 2450 20050 2700
 Connection ~ 20050 2700
-Wire Wire Line
-	20050 2700 20200 2700
 Text GLabel 19900 3850 2    50   Input ~ 0
 VDD
@@
 L Device:CP C29
 U 1 1 5EEDF346
-P 8700 5800
-F 0 "C29" H 8818 5846 50  0000 L CNN
-F 1 "10uF" H 8818 5755 50  0000 L CNN
-F 2 "Capacitor_SMD:CP_Elec_5x5.3" H 8738 5650 50  0001 C CNN
-F 3 "~" H 8700 5800 50  0001 C CNN
-	1    8700 5800
+P 8300 5800
+F 0 "C29" H 8418 5846 50  0000 L CNN
+F 1 "10uF" H 8418 5755 50  0000 L CNN
+F 2 "Capacitor_SMD:CP_Elec_5x5.3" H 8338 5650 50  0001 C CNN
+F 3 "~" H 8300 5800 50  0001 C CNN
+	1    8300 5800
 	0    1    1    0
 $EndComp
@@
 	7550 5800 7200 5800
 Wire Wire Line
-	8550 5800 8100 5800
+	8150 5800 8100 5800
 Wire Wire Line
 	7550 6400 7550 6550
@@
 Text GLabel 4500 6800 1    50   Input ~ 0
 scaled_input
-Text GLabel 9250 5800 2    50   Input ~ 0
+Text GLabel 8650 5800 2    50   Input ~ 0
 output
 $Comp
@@
 Wire Wire Line
 	7550 13700 7550 13950
-$Comp
-L Device:C C20
-U 1 1 5F362F56
-P 6200 13200
-F 0 "C20" V 5948 13200 50  0000 C CNN
-F 1 "560uF" V 6039 13200 50  0000 C CNN
-F 2 "Capacitor_SMD:C_0603_1608Metric" H 6238 13050 50  0001 C CNN
-F 3 "~" H 6200 13200 50  0001 C CNN
-	1    6200 13200
-	-1   0    0    1
-$EndComp
 Wire Wire Line
 	6450 13050 6200 13050
-Wire Wire Line
-	6200 13350 6200 13400
-Wire Wire Line
-	6200 13400 6450 13400
 Wire Wire Line
 	6200 11600 6200 13050
@@
 Wire Wire Line
 	6200 11600 6400 11600
-Connection ~ 6200 13050
 Wire Wire Line
 	5500 11900 6000 11900
 Wire Wire Line
 	6000 11900 6000 13400
-Wire Wire Line
-	6000 13400 6200 13400
 Connection ~ 5500 11900
-Connection ~ 6200 13400
 Wire Wire Line
 	5500 12000 5850 12000
@@
 	1    0    0    -1
 $EndComp
-Connection ~ 20200 2700
 $Comp
 L Device:R R36
@@
 	-1   0    0    1
 $EndComp
-Wire Wire Line
-	20200 2900 20200 2700
 Wire Wire Line
 	20200 3600 20200 3500
@@
 Text Notes 13550 1700 0    158  ~ 32
 POWER SUPPLY\n
-$Comp
-L Switch:SW_SPDT SW1
-U 1 1 5FB4A7F8
-P 9200 5000
-F 0 "SW1" H 9200 4675 50  0000 C CNN
-F 1 "SW_SPDT" H 9200 4766 50  0000 C CNN
-F 2 "Connector:FanPinHeader_1x03_P2.54mm_Vertical" H 9200 5000 50  0001 C CNN
-F 3 "~" H 9200 5000 50  0001 C CNN
-	1    9200 5000
-	-1   0    0    1
-$EndComp
-Wire Wire Line
-	8850 5800 8950 5800
-Wire Wire Line
-	9000 5100 8950 5100
-Wire Wire Line
-	8950 5100 8950 5800
-Connection ~ 8950 5800
-Wire Wire Line
-	8950 5800 9250 5800
+Wire Wire Line
+	8450 5800 8550 5800
+Wire Wire Line
+	9000 5100 8550 5100
+Wire Wire Line
+	8550 5100 8550 5800
+Connection ~ 8550 5800
+Wire Wire Line
+	8550 5800 8650 5800
 Wire Wire Line
 	8900 4900 9000 4900
@@
 Wire Wire Line
 	20900 3200 20900 3450
-Wire Wire Line
-	20200 2700 20450 2700
 $Comp
 L Connector:AudioJack2 J4
@@
 	-1   0    0    1
 $EndComp
+$Comp
+L Switch:SW_DPDT_x2 SW1
+U 1 1 5EC2108A
+P 9200 5000
+F 0 "SW1" H 9200 4675 50  0000 C CNN
+F 1 "SW_DPDT_x2" H 9200 4766 50  0000 C CNN
+F 2 "M2028B2B1W03:M2028B2B1W03" H 9200 5000 50  0001 C CNN
+F 3 "~" H 9200 5000 50  0001 C CNN
+	1    9200 5000
+	-1   0    0    1
+$EndComp
+Wire Wire Line
+	9000 6200 9150 6200
+$Comp
+L Device:LED D9
+U 1 1 5EC289FC
+P 9750 6750
+F 0 "D9" V 9789 6633 50  0000 R CNN
+F 1 "LED" V 9698 6633 50  0000 R CNN
+F 2 "LED_SMD:LED_1206_3216Metric" H 9750 6750 50  0001 C CNN
+F 3 "~" H 9750 6750 50  0001 C CNN
+	1    9750 6750
+	0    -1   -1   0
+$EndComp
+$Comp
+L power:GND #PWR037
+U 1 1 5EC28A02
+P 9750 7000
+F 0 "#PWR037" H 9750 6750 50  0001 C CNN
+F 1 "GND" H 9755 6827 50  0000 C CNN
+F 2 "" H 9750 7000 50  0001 C CNN
+F 3 "" H 9750 7000 50  0001 C CNN
+	1    9750 7000
+	1    0    0    -1
+$EndComp
+$Comp
+L Device:R R39
+U 1 1 5EC28A09
+P 9750 6450
+F 0 "R39" H 9820 6496 50  0000 L CNN
+F 1 "470" H 9820 6405 50  0000 L CNN
+F 2 "Resistor_SMD:R_0603_1608Metric" V 9680 6450 50  0001 C CNN
+F 3 "~" H 9750 6450 50  0001 C CNN
+	1    9750 6450
+	-1   0    0    1
+$EndComp
+Wire Wire Line
+	9750 6300 9750 6100
+Wire Wire Line
+	9750 7000 9750 6900
+Text GLabel 9000 6200 0    50   Input ~ 0
+VCC
+$Comp
+L Switch:SW_DPDT_x2 SW1
+U 2 1 5EC232A2
+P 9350 6100
+F 0 "SW1" V 9304 6248 50  0000 L CNN
+F 1 "SW_DPDT_x2" V 9395 6248 50  0000 L CNN
+F 2 "M2028B2B1W03:M2028B2B1W03" H 9350 6100 50  0001 C CNN
+F 3 "~" H 9350 6100 50  0001 C CNN
+	2    9350 6100
+	-1   0    0    1
+$EndComp
+Wire Wire Line
+	9550 6100 9750 6100
+Wire Wire Line
+	20200 2700 20450 2700
+Wire Wire Line
+	20050 2700 20200 2700
+Connection ~ 20200 2700
+Wire Wire Line
+	20200 2900 20200 2700
+Wire Wire Line
+	6000 13400 6450 13400
 $EndSCHEMATC

Commit message: Autorouting done
Parts:
- added H1, H2, H3, H4: MountingHole, MountingHole:MountingHole_3mm, symbol Mechanical:MountingHole
- added U7: logo, imgs:ratatech_bitmap, symbol logo:logo
Connections:
- net VDD: now also Q2.3 (C); no longer Q2.1 (E)
- net at R21.1: now also Q2.1 (E); no longer Q2.3 (C)
Other:
- moved on the sheet: C1, C10, C11, C12, C13, C14, C15, C16, C17, C18, C19, C2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

Commit message: Added mouser part numbers
Parts:
- C1, C10, C11, C16, C17, C3, C7: Mouser Part Number (none) -> 710-885012206071
- C12, C13, C19, C23, C25, C29, C33, C38, C4, C9: Mouser Part Number (none) -> 598-AVE106M35C12T-F
- C14, C15: Mouser Part Number (none) -> 80-C0603C561G8HACTU
- C18, C26: Mouser Part Number (none) -> 603-C0603KRX7R9BB392
- C2, C22: Mouser Part Number (none) -> 710-885012206040
- C21, C24: Mouser Part Number (none) -> 555-RVS-35V4R7MU-R
- C27, C28, C30, C31, C35, C5: Mouser Part Number (none) -> 661-EMZJ6R3A101ME61G
- C32, C36, C37: Mouser Part Number (none) -> 555-RVS-50V2R2MU-R
- C34: Mouser Part Number (none) -> 603-CC603KRX7R9BB202
- C39, C40: Mouser Part Number (none) -> 555-RVS-50VR47MU-R
- C6: Mouser Part Number (none) -> 140-VE470M1CTR0505
- C8: Mouser Part Number (none) -> 710-885012206081
- D1, D2, D3, D5, D6: Mouser Part Number (none) -> 621-MMBD4148-F
- D4, D8, D9: Mouser Part Number (none) -> 327-BR1101WTR
- D7: Mouser Part Number (none) -> 863-SZMM3Z6V8ST1G
- J1, J4: Mouser Part Number (none) -> 550-10284G
- J2, J3: Mouser Part Number (none) -> 474-PRT-09749
- J5: Mouser Part Number (none) -> 490-PJ-102BH
- Q1, Q3: Mouser Part Number (none) -> 583-MMBT4401
- Q2, Q4: Mouser Part Number (none) -> 583-MMBT3906
- R1, R22: Mouser Part Number (none) -> 71-CRCW06034K70JNEAC
- R10: Mouser Part Number (none) -> 71-CRCW06033K30FKEAC
- R11, R5: Mouser Part Number (none) -> 71-CRCW0603560RFKEAC
- R12, R31, R6, R7: Mouser Part Number (none) -> 71-CRCW060322K0FKEAC
- R13, R14: Mouser Part Number (none) -> 652-CR0603-FX3901ELF
- R15, R16, R17, R18, R24, R25, R28, R29, R33, R35: Mouser Part Number (none) -> 755-SFR03EZPF1002
- R19, R23: Mouser Part Number (none) -> 603-RC0603FR-0715KL
- R2: Mouser Part Number (none) -> 603-RC0603FR-10220KL
- R20, R21: Mouser Part Number (none) -> 71-CRCW060310R0FKEAC
- R26: Mouser Part Number (none) -> 652-CR0603JW-562ELF
- R27, R3, R34: Mouser Part Number (none) -> 71-CRCW0603100KFKEAC
- R30: Mouser Part Number (none) -> 71-CRCW0603100RFKEAC
- R32: Mouser Part Number (none) -> 652-CR0603FX-2403ELF
- R36, R39: Mouser Part Number (none) -> 71-CRCW0603470RFKEAC
- R37: Mouser Part Number (none) -> 71-CRCW06031K00FKEAC
- R38: Mouser Part Number (none) -> 652-CR0603FX-2700ELF
- R4: Mouser Part Number (none) -> 71-CRCW0603220RFKEAC
- R8: Mouser Part Number (none) -> 71-CRCW0603680RJNEAC
- R9: Mouser Part Number (none) -> 71-CRCW0603150RJNEAC
- RV1: Mouser Part Number (none) -> RK09D113AF25A15
- RV2: Mouser Part Number (none) -> 652-PTV09A-4030UB203
- RV3, RV4: Mouser Part Number (none) -> 688-RK09D113000Q
- RV5: Mouser Part Number (none) -> 688-RK09D113000K
- SW1: Mouser Part Number (none) -> 612-100-F1121
- SW2: Mouser Part Number (none) -> 611-OS102011MA1QN1
- U1, U2: Mouser Part Number (none) -> 595-NE5532DR
- U3: Mouser Part Number (none) -> 200-ICF308TO
- U4: Mouser Part Number (none) -> 595-LT1054CDWR
- U5: Mouser Part Number (none) -> 511-L78M12CDT-TR
- U6: Mouser Part Number (none) -> 512-KA79M12RTF

Commit message: Finished BOM with mouser part numbers
Parts:
- C21, C24: Mouser Part Number 555-RVS-35V4R7MU-R -> 647-UWT1H4R7MCL1B
- C32, C36, C37: Mouser Part Number 555-RVS-50V2R2MU-R -> 661-EMVE630ADA3R3ME5
- C39, C40: Mouser Part Number 555-RVS-50VR47MU-R -> RVS-50V010MU-R
- Q1, Q3: Mouser Part Number 583-MMBT4401 -> 771-MMBT3904T/R
- Q2, Q4: Mouser Part Number 583-MMBT3906 -> 771-MMBT3906T/R
- RV1: Mouser Part Number RK09D113AF25A15 -> 652-PTV09A4025FB104
- RV3, RV4: Mouser Part Number 688-RK09D113000Q -> 652-PTV09A-4025FB103
- RV5: Mouser Part Number 688-RK09D113000K -> 652-PTV09A-4225FA503
- SW1: Mouser Part Number 612-100-F1121 -> 612-100DP3T4B1M1Q
Changed lines of the file:
@@
 F 2 "Capacitor_SMD:CP_Elec_5x5.3" H 14538 3700 50  0001 C CNN
 F 3 "~" H 14500 3850 50  0001 C CNN
-F 4 "555-RVS-50V2R2MU-R" H 14500 3850 50  0001 C CNN "Mouser Part Number"
+F 4 "661-EMVE630ADA3R3ME5" H 14500 3850 50  0001 C CNN "Mouser Part Number"
 	1    14500 3850
 	1    0    0    -1
@@
 F 2 "Capacitor_SMD:CP_Elec_5x5.3" H 18188 2500 50  0001 C CNN
 F 3 "~" H 18150 2650 50  0001 C CNN
-F 4 "555-RVS-50V2R2MU-R" H 18150 2650 50  0001 C CNN "Mouser Part Number"
+F 4 "661-EMVE630ADA3R3ME5" H 18150 2650 50  0001 C CNN "Mouser Part Number"
 	1    18150 2650
 	1    0    0    -1
@@
 F 2 "Capacitor_SMD:CP_Elec_5x5.3" H 19138 2500 50  0001 C CNN
 F 3 "~" H 19100 2650 50  0001 C CNN
-F 4 "555-RVS-50VR47MU-R " H 19100 2650 50  0001 C CNN "Mouser Part Number"
+F 4 "RVS-50V010MU-R" H 19100 2650 50  0001 C CNN "Mouser Part Number"
 	1    19100 2650
 	1    0    0    -1
@@
 F 2 "Capacitor_SMD:CP_Elec_5x5.3" H 18188 3700 50  0001 C CNN
 F 3 "~" H 18150 3850 50  0001 C CNN
-F 4 "555-RVS-50V2R2MU-R" H 18150 3850 50  0001 C CNN "Mouser Part Number"
+F 4 "661-EMVE630ADA3R3ME5" H 18150 3850 50  0001 C CNN "Mouser Part Number"
 	1    18150 3850
 	-1   0    0    1
@@
 F 2 "Capacitor_SMD:CP_Elec_5x5.3" H 19138 3700 50  0001 C CNN
 F 3 "~" H 19100 3850 50  0001 C CNN
-F 4 "555-RVS-50VR47MU-R " H 19100 3850 50  0001 C CNN "Mouser Part Number"
+F 4 "RVS-50V010MU-R" H 19100 3850 50  0001 C CNN "Mouser Part Number"
 	1    19100 3850
 	-1   0    0    1
@@
 F 2 "Potentiometer_THT:Potentiometer_Alps_RK09K_Single_Vertical" H 6300 6300 50  0001 C CNN
 F 3 "~" H 6300 6300 50  0001 C CNN
-F 4 "688-RK09D113000Q" H 6300 6300 50  0001 C CNN "Mouser Part Number"
+F 4 "652-PTV09A-4025FB103" H 6300 6300 50  0001 C CNN "Mouser Part Number"
 	1    6300 6300
 	1    0    0    -1
@@
 F 2 "Potentiometer_THT:Potentiometer_Alps_RK09K_Single_Vertical" H 4950 7550 50  0001 C CNN
 F 3 "~" H 4950 7550 50  0001 C CNN
-F 4 "688-RK09D113000Q" H 4950 7550 50  0001 C CNN "Mouser Part Number"
+F 4 "652-PTV09A-4025FB103" H 4950 7550 50  0001 C CNN "Mouser Part Number"
 	1    4950 7550
 	1    0    0    -1
@@
 F 2 "Capacitor_SMD:CP_Elec_5x5.3" H 7338 10350 50  0001 C CNN
 F 3 "~" H 7300 10500 50  0001 C CNN
-F 4 "555-RVS-35V4R7MU-R" H 7300 10500 50  0001 C CNN "Mouser Part Number"
+F 4 "647-UWT1H4R7MCL1B " H 7300 10500 50  0001 C CNN "Mouser Part Number"
 	1    7300 10500
 	0    -1   -1   0
@@
 F 2 "Potentiometer_THT:Potentiometer_Alps_RK09K_Single_Vertical" H 7900 12650 50  0001 C CNN
 F 3 "~" H 7900 12650 50  0001 C CNN
-F 4 "688-RK09D113000K" H 7900 12650 50  0001 C CNN "Mouser Part Number"
+F 4 "652-PTV09A-4225FA503" H 7900 12650 50  0001 C CNN "Mouser Part Number"
 	1    7900 12650
 	1    0    0    -1
@@
 F 2 "Capacitor_SMD:CP_Elec_5x5.3" H 7438 11150 50  0001 C CNN
 F 3 "~" H 7400 11300 50  0001 C CNN
-F 4 "555-RVS-35V4R7MU-R" H 7400 11300 50  0001 C CNN "Mouser Part Number"
+F 4 "647-UWT1H4R7MCL1B " H 7400 11300 50  0001 C CNN "Mouser Part Number"
 	1    7400 11300
 	0    -1   -1   0
@@
 F 2 "Package_TO_SOT_SMD:SOT-23" H 7050 3925 50  0001 L CIN
 F 3 "https://www.fairchildsemi.com/datasheets/2N/2N3906.pdf" H 6850 4000 50  0001 L CNN
-F 4 "583-MMBT3906" H 6850 4000 50  0001 C CNN "Mouser Part Number"
+F 4 "771-MMBT3906T/R" H 6850 4000 50  0001 C CNN "Mouser Part Number"
 	1    6850 4000
 	1    0    0    1
@@
 F 2 "Package_TO_SOT_SMD:SOT-23" H 7050 2625 50  0001 L CIN
 F 3 "https://www.fairchildsemi.com/datasheets/2N/2N3904.pdf" H 6850 2700 50  0001 L CNN
-F 4 "583-MMBT4401" H 6850 2700 50  0001 C CNN "Mouser Part Number"
+F 4 "771-MMBT3904T/R" H 6850 2700 50  0001 C CNN "Mouser Part Number"
 	1    6850 2700
 	1    0    0    -1
@@
 F 2 "Package_TO_SOT_SMD:SOT-23" H 18600 7375 50  0001 L CIN
 F 3 "https://www.fairchildsemi.com/datasheets/2N/2N3904.pdf" H 18400 7450 50  0001 L CNN
-F 4 "583-MMBT4401" H 18400 7450 50  0001 C CNN "Mouser Part Number"
+F 4 "771-MMBT3904T/R" H 18400 7450 50  0001 C CNN "Mouser Part Number"
 	1    18400 7450
 	1    0    0    -1
@@
 F 2 "Package_TO_SOT_SMD:SOT-23" H 20000 7625 50  0001 L CIN
 F 3 "https://www.fairchildsemi.com/datasheets/2N/2N3906.pdf" H 19800 7700 50  0001 L CNN
-F 4 "583-MMBT3906" H 19800 7700 50  0001 C CNN "Mouser Part Number"
+F 4 "771-MMBT3906T/R" H 19800 7700 50  0001 C CNN "Mouser Part Number"
 	1    19800 7700
 	1    0    0    1
@@
 F 2 "Potentiometer_THT:Potentiometer_Alps_RK09K_Single_Vertical" H 2150 3750 50  0001 C CNN
 F 3 "~" H 2150 3750 50  0001 C CNN
-F 4 "RK09D113AF25A15 " H 2150 3750 50  0001 C CNN "Mouser Part Number"
+F 4 "652-PTV09A4025FB104" H 2150 3750 50  0001 C CNN "Mouser Part Number"
 	1    2150 3750
 	0    1    1    0
@@
 F 2 "M2028B2B1W03:M2028B2B1W03" H 9650 5400 50  0001 C CNN
 F 3 "~" H 9650 5400 50  0001 C CNN
-F 4 " 612-100-F1121" H 9650 5400 50  0001 C CNN "Mouser Part Number"
+F 4 "612-100DP3T4B1M1Q" H 9650 5400 50  0001 C CNN "Mouser Part Number"
 	1    9650 5400
 	-1   0    0    1
@@
 F 2 "M2028B2B1W03:M2028B2B1W03" H 9800 6500 50  0001 C CNN
 F 3 "~" H 9800 6500 50  0001 C CNN
-F 4 " 612-100-F1121" H 9800 6500 50  0001 C CNN "Mouser Part Number"
+F 4 "612-100DP3T4B1M1Q" H 9800 6500 50  0001 C CNN "Mouser Part Number"
 	2    9800 6500
 	-1   0    0    1
